File: TX/Schaltplan_TX/schimmeliger_keller.sch (EAGLE design)
At the start: 8 parts, among them IC1 LoRa Module, Q1 2N3904, U1 LOPY4

Commit message: fast fertig
Parts:
- added R2: 4.7k, eagle-ltspice:R0204/7
- B1: value 3V (2x AA) -> 4,5V (3x AAA)
Connections:
- net N$3: now also R2.1
- net VDD: now also R2.2
Changed lines of the file:
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@@
 <part name="FRAME1" library="frames" deviceset="A5L-LOC" device=""/>
 <part name="ANT1" library="discrete" deviceset="ANTENNA" device=""/>
-<part name="B1" library="battery" deviceset="AB9V" device="" value="3V (2x AA)"/>
+<part name="B1" library="battery" deviceset="AB9V" device="" value="4,5V (3x AAA)"/>
 <part name="SENS1" library="pinhead" deviceset="PINHD-1X3" device=""/>
 <part name="GND1" library="supply1" deviceset="GND" device=""/>
@@
 <part name="IC1" library="blubb" deviceset="U893BSE" device="" value="LoRa Module"/>
 <part name="R1" library="eagle-ltspice" deviceset="R" device="0204/7" value="1k"/>
+<part name="R2" library="eagle-ltspice" deviceset="R" device="0204/7" value="4.7k"/>
+<part name="SUPPLY5" library="supply2" deviceset="VDD" device=""/>
 </parts>
 <sheets>
@@
 </instance>
 <instance part="R1" gate="G$1" x="111.76" y="45.72"/>
+<instance part="R2" gate="G$1" x="-7.62" y="60.96" rot="R90"/>
+<instance part="SUPPLY5" gate="G$1" x="-7.62" y="71.12"/>
 </instances>
 <busses>
@@
 <wire x1="50.8" y1="81.28" x2="55.88" y2="81.28" width="0.1524" layer="91"/>
 </segment>
+<segment>
+<pinref part="SUPPLY5" gate="G$1" pin="VDD"/>
+<pinref part="R2" gate="G$1" pin="2"/>
+<wire x1="-7.62" y1="68.58" x2="-7.62" y2="66.04" width="0.1524" layer="91"/>
+</segment>
 </net>
 <net name="N$8" class="0">
@@
 <pinref part="U1" gate="G$1" pin="P9"/>
 <pinref part="SENS1" gate="A" pin="2"/>
-<wire x1="55.88" y1="48.26" x2="-15.24" y2="48.26" width="0.1524" layer="91"/>
+<wire x1="55.88" y1="48.26" x2="-7.62" y2="48.26" width="0.1524" layer="91"/>
+<wire x1="-7.62" y1="48.26" x2="-15.24" y2="48.26" width="0.1524" layer="91"/>
 <wire x1="-15.24" y1="48.26" x2="-15.24" y2="93.98" width="0.1524" layer="91"/>
+<pinref part="R2" gate="G$1" pin="1"/>
+<wire x1="-7.62" y1="55.88" x2="-7.62" y2="48.26" width="0.1524" layer="91"/>
+<junction x="-7.62" y="48.26"/>
 </segment>
 </net>

Commit message: fertich
Connections:
- net N$2: now also R2.2
- net VDD: no longer R2.2
Other:
- moved on the sheet: R2
Changed lines of the file:
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@@
 <part name="R1" library="eagle-ltspice" deviceset="R" device="0204/7" value="1k"/>
 <part name="R2" library="eagle-ltspice" deviceset="R" device="0204/7" value="4.7k"/>
-<part name="SUPPLY5" library="supply2" deviceset="VDD" device=""/>
 </parts>
 <sheets>
@@
 </instance>
 <instance part="R1" gate="G$1" x="111.76" y="45.72"/>
-<instance part="R2" gate="G$1" x="-7.62" y="60.96" rot="R90"/>
-<instance part="SUPPLY5" gate="G$1" x="-7.62" y="71.12"/>
+<instance part="R2" gate="G$1" x="-7.62" y="33.02" rot="R270"/>
 </instances>
 <busses>
@@
 <pinref part="Q1" gate="G1" pin="E"/>
 <wire x1="127" y1="40.64" x2="127" y2="20.32" width="0.1524" layer="91"/>
-<wire x1="127" y1="20.32" x2="-17.78" y2="20.32" width="0.1524" layer="91"/>
+<wire x1="127" y1="20.32" x2="-7.62" y2="20.32" width="0.1524" layer="91"/>
 <pinref part="SENS1" gate="A" pin="1"/>
+<wire x1="-7.62" y1="20.32" x2="-17.78" y2="20.32" width="0.1524" layer="91"/>
 <wire x1="-17.78" y1="20.32" x2="-17.78" y2="93.98" width="0.1524" layer="91"/>
+<pinref part="R2" gate="G$1" pin="2"/>
+<wire x1="-7.62" y1="27.94" x2="-7.62" y2="20.32" width="0.1524" layer="91"/>
+<junction x="-7.62" y="20.32"/>
 </segment>
 </net>
@@
 <wire x1="50.8" y1="81.28" x2="55.88" y2="81.28" width="0.1524" layer="91"/>
 </segment>
-<segment>
-<pinref part="SUPPLY5" gate="G$1" pin="VDD"/>
-<pinref part="R2" gate="G$1" pin="2"/>
-<wire x1="-7.62" y1="68.58" x2="-7.62" y2="66.04" width="0.1524" layer="91"/>
-</segment>
 </net>
 <net name="N$8" class="0">
@@
 <wire x1="-15.24" y1="48.26" x2="-15.24" y2="93.98" width="0.1524" layer="91"/>
 <pinref part="R2" gate="G$1" pin="1"/>
-<wire x1="-7.62" y1="55.88" x2="-7.62" y2="48.26" width="0.1524" layer="91"/>
+<wire x1="-7.62" y1="38.1" x2="-7.62" y2="48.26" width="0.1524" layer="91"/>
 <junction x="-7.62" y="48.26"/>
 </segment>
